Commit message: joint camera

File: src/rosbot_description/urdf/rosbot.xacro (robot description, xacro)
@@ -236,5 +236,5 @@
   </transmission>
   <!-- Orbbec Astra RGBD Camera -->
-  <joint name="astra_joint" type="fixed">
+  <joint name="astra_joint" type="continuous">
     <axis xyz="0 0 0" />
     <origin xyz="-0.03 0 0.18" rpy="0 0 0"/>

Commit message: joint camera fix

File: src/rosbot_description/urdf/rosbot.xacro (robot description, xacro)
@@ -237,8 +237,10 @@
   <!-- Orbbec Astra RGBD Camera -->
   <joint name="astra_joint" type="continuous">
-    <axis xyz="0 0 0" />
+    <axis xyz="0 0 1" />
     <origin xyz="-0.03 0 0.18" rpy="0 0 0"/>
     <parent link="body_link"/>
     <child link="camera_link"/>
+    <limit effort="1" velocity="10"/>
+    <joint_properties damping="5.0" friction="1.0"/>
   </joint>
   <link name="camera_link">

Commit message: transmission camera

File: src/rosbot_description/urdf/rosbot.xacro (robot description, xacro)
@@ -244,4 +244,13 @@
     <joint_properties damping="5.0" friction="1.0"/>
   </joint>
+  <transmission name="astra_joint_trans" type="SimpleTransmission">
+    <type>transmission_interface/SimpleTransmission</type>
+    <actuator name="astra_joint_motor">
+      <mechanicalReduction>1</mechanicalReduction>
+    </actuator>
+    <joint name="astra_joint">
+      <hardwareInterface>hardware_interface/EffortJointInterface</hardwareInterface>
+    </joint>
+  </transmission>
   <link name="camera_link">
     <collision>
